File: core-components/korry/Korry.kicad_sch (KiCad schematic)
At the start: 11 parts, among them J1 Conn_01x02_Pin, J2 Conn_01x04_Pin

Commit message: Korry V3
Korry V3
Parts:
- removed D2, D3: LED, LED_THT:LED_D3.0mm, symbol Device:LED
- removed R1, R3: R, Resistor_SMD:R_1210_3225Metric_Pad1.30x2.65mm_HandSolder, symbol Device:R
Connections:
- net at J2.3 (Pin_3): now also R4.2; no longer D4.2 (A)
- net at J2.4 (Pin_4): now also D4.2 (A); no longer R4.2
Other:
- moved on the sheet: D1, D4, R2, R4
