File: core-components/korry/Korry.kicad_pcb (KiCad board)
At the start: 2 copper layers, 173.7 x 105 mm, 184 parts, among them J1 Conn_01x02_Pin, J2 Conn_01x04_Pin

Commit message: Korry V3
Korry V3
Parts:
- removed the D1 at (139.1, 79.4)
- removed the D1 at (162.5, 102.9)
- removed the D1 at (186.0, 79.4)
- removed the D1 at (115.6, 79.4)
- removed the D1 at (115.6, 102.9)
- removed the D1 at (186.0, 32.4)
- removed the D1 at (139.1, 32.4)
- removed the D1 at (162.5, 32.4)
- removed the D1 at (186.0, 102.9)
- removed the D1 at (115.6, 32.4)
- removed the D1 at (139.1, 55.9)
- removed the D1 at (115.6, 55.9)
- removed the D1 at (139.1, 102.9)
- removed the D1 at (186.0, 55.9)
- removed the D1 at (162.5, 55.9)
- removed the D1 at (162.5, 79.4)
- removed the D2 at (108.6, 55.9)
- removed the D2 at (108.6, 102.9)
- removed the D2 at (155.5, 79.4)
- removed the D2 at (108.6, 32.4)
- removed the D2 at (132.1, 102.9)
- removed the D2 at (132.1, 32.4)
- removed the D2 at (132.1, 55.9)
- removed the D2 at (179.0, 32.4)
- removed the D2 at (155.5, 32.4)
- removed the D2 at (155.5, 102.9)
- removed the D2 at (155.5, 55.9)
- removed the D2 at (108.6, 79.4)
- removed the D2 at (179.0, 55.9)
- removed the D2 at (179.0, 102.9)
- removed the D2 at (132.1, 79.4)
- removed the D2 at (179.0, 79.4)
- removed D3 (x16), D4 (x16): LED, LED_THT:LED_D3.0mm
- removed the J1 at (175.8, 85.5)
- removed the J1 at (128.9, 62.0)
- removed the J1 at (105.5, 38.5)
- removed the J1 at (175.8, 38.5)
- removed the J1 at (152.4, 85.5)
- removed the J1 at (128.9, 85.5)
- removed the J1 at (105.5, 109.0)
- removed the J1 at (152.4, 109.0)
- removed the J1 at (152.4, 62.0)
- removed the J1 at (175.8, 62.0)
- removed the J1 at (152.4, 38.5)
- removed the J1 at (128.9, 109.0)
- removed the J1 at (105.5, 62.0)
- removed the J1 at (105.5, 85.5)
- removed the J1 at (128.9, 38.5)
- removed the J1 at (175.8, 109.0)
- removed the J2 at (144.5, 31.5)
- removed the J2 at (121.0, 31.5)
- removed the J2 at (121.0, 55.0)
- removed the J2 at (121.0, 78.5)
- removed the J2 at (121.0, 102.0)
- removed the J2 at (168.0, 31.5)
- removed the J2 at (191.4, 78.5)
- removed the J2 at (191.4, 102.0)
- removed the J2 at (168.0, 78.5)
- removed the J2 at (144.5, 78.5)
- removed the J2 at (191.4, 55.0)
- removed the J2 at (144.5, 55.0)
- removed the J2 at (168.0, 55.0)
- removed the J2 at (168.0, 102.0)
- removed the J2 at (144.5, 102.0)
- removed the J2 at (191.4, 31.5)
- removed the R1 at (132.1, 100.2)
- removed the R1 at (155.5, 29.7)
- removed the R1 at (108.6, 53.2)
- removed the R1 at (132.1, 29.7)
- removed the R1 at (179.0, 76.7)
- removed the R1 at (108.6, 29.7)
- removed the R1 at (132.1, 76.7)
- removed the R1 at (108.6, 100.2)
- removed the R1 at (132.1, 53.2)
- removed the R1 at (155.5, 53.2)
- removed the R1 at (179.0, 100.2)
- removed the R1 at (179.0, 29.7)
- removed the R1 at (179.0, 53.2)
- removed the R1 at (155.5, 100.2)
- removed the R1 at (108.6, 76.7)
- removed the R1 at (155.5, 76.7)
- removed the R2 at (187.1, 76.7)
- removed the R2 at (163.6, 53.2)
- removed the R2 at (187.1, 29.7)
- removed the R2 at (163.6, 29.7)
- removed the R2 at (116.7, 76.7)
- removed the R2 at (163.6, 76.7)
- removed the R2 at (140.2, 53.2)
- removed the R2 at (163.6, 100.2)
- removed the R2 at (116.7, 29.7)
- removed the R2 at (187.1, 100.2)
- removed the R2 at (187.1, 53.2)
- removed the R2 at (116.7, 53.2)
- removed the R2 at (140.2, 76.7)
- removed the R2 at (140.2, 100.2)
- removed the R2 at (140.2, 29.7)
- removed the R2 at (116.7, 100.2)
- removed R3 (x16), R4 (x16): R, Resistor_SMD:R_1210_3225Metric_Pad1.30x2.65mm_HandSolder
- removed REF** (x8): LED_D5.0mm, LED_THT:LED_D5.0mm
- removed the U1 at (142.6, 64.8)
- removed the U1 at (142.6, 41.3)
- removed the U1 at (166.0, 88.3)
- removed the U1 at (119.1, 64.8)
- removed the U1 at (166.0, 64.8)
- removed the U1 at (166.0, 111.8)
- removed the U1 at (142.6, 111.8)
- removed the U1 at (142.6, 88.3)
- removed the U1 at (189.5, 88.3)
- removed the U1 at (189.5, 64.8)
- removed the U1 at (189.5, 41.3)
- removed the U1 at (166.0, 41.3)
- removed the U1 at (189.5, 111.8)
- removed the U1 at (119.1, 88.3)
- removed the U1 at (119.1, 41.3)
- removed the U1 at (119.1, 111.8)
- added D1: LED, LED_THT:LED_D3.0mm, F.Cu at (134.1, 83.9)
- added D2: LED, LED_THT:LED_D3.0mm, F.Cu at (134.2, 72.9)
- added J1: Conn_01x02_Pin, Connector_PinHeader_2.54mm:PinHeader_1x02_P2.54mm_Vertical, B.Cu at (128.2, 82.8)
- added J2: Conn_01x04_Pin, Connector_PinHeader_2.54mm:PinHeader_1x04_P2.54mm_Vertical, B.Cu at (128.2, 71.3)
- added R1: R, Resistor_SMD:R_1210_3225Metric_Pad1.30x2.65mm_HandSolder, F.Cu at (140.6, 85.5)
- added R2: R, Resistor_SMD:R_1210_3225Metric_Pad1.30x2.65mm_HandSolder, F.Cu at (140.7, 71.4)
- added U1: ~, OpenA3XX:Korry_Switch_Discrete, F.Cu at (141.4, 82.5)
Routing:
- net Net-(J2-Pin_2): track 0.00 -> 27.3 mm, vias 0 -> 1
- net Net-(D1-A): track 0.00 -> 26.5 mm
- net Board_14-Net-(J2-Pin_2): track 21.9 -> 0.00 mm
- net Board_10-Net-(J2-Pin_2): track 21.9 -> 0.00 mm
- net Board_8-Net-(J2-Pin_2): track 21.9 -> 0.00 mm
- net Board_6-Net-(J2-Pin_2): track 21.9 -> 0.00 mm
- net Board_2-Net-(J2-Pin_2): track 21.9 -> 0.00 mm
- net Board_12-Net-(J2-Pin_2): track 21.9 -> 0.00 mm
- net Board_4-Net-(J2-Pin_2): track 21.9 -> 0.00 mm
- net Board_13-Net-(J2-Pin_2): track 21.9 -> 0.00 mm
- net Board_0-Net-(J2-Pin_2): track 21.9 -> 0.00 mm
- net Board_9-Net-(J2-Pin_2): track 21.9 -> 0.00 mm
- net Board_5-Net-(J2-Pin_2): track 21.9 -> 0.00 mm
- net Board_1-Net-(J2-Pin_2): track 21.9 -> 0.00 mm
- net Board_11-Net-(J2-Pin_2): track 21.9 -> 0.00 mm
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Other:
- board size 173.7 x 105 mm -> 18.5 x 18.6 mm
- board text removed: "+"
- board text removed: "1"
- board text removed: "MANTOGA"
- board text removed: "OPENA3XX"
- board text removed: "SW"

Commit message: KorryUpdates
KorryUpdates
Parts:
- added G***: LOGO, OpenA3XX:OpenA3XXLogoSmall, B.Cu at (135.6, 78.2)
